File: public/sample-sensor.kicad_pcb (KiCad board)
At the start: 2 copper layers, 64 x 39 mm, 2 parts, among them J1 SENSOR, J2 CONTROLLER

Commit message: test: gate auto-layout with KiCad DRC
Parts:
- J1, J2: footprint Connector_PinHeader_2.54mm:PinHeader_1x04_P2.54mm_Vertical -> Copperline_SensorHeader_1x04_P9mm_Vertical
Changed lines of the file:
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@@
   (net 3 "SENSOR_CLOCK")
   (net 4 "SENSOR_GND")
-  (footprint "Connector_PinHeader_2.54mm:PinHeader_1x04_P2.54mm_Vertical"
+  (footprint "Copperline_SensorHeader_1x04_P9mm_Vertical"
     (layer "F.Cu")
     (at 18 20)
@@
     (pad "4" thru_hole circle (at 0 27) (size 3.6 3.6) (drill 1.2) (layers "*.Cu" "*.Mask") (net 4 "SENSOR_GND"))
   )
-  (footprint "Connector_PinHeader_2.54mm:PinHeader_1x04_P2.54mm_Vertical"
+  (footprint "Copperline_SensorHeader_1x04_P9mm_Vertical"
     (layer "F.Cu")
     (at 66 20)
